File: eagle/proto.sch (EAGLE design)
At the start: 15 parts, among them J1 DCJ0202, X1 NRF51822-RIGHT

Commit message: eagle: Kolejna wersja prototypu
Signed-off-by: Pawel Szewczyk <pfpawelec@gmail.com>
Parts:
- added DEC+, DEC-, RA+, RA-: TACT-SWITCH, eq-custom2:TACT-SWITCH
- added LED3, LED4: (no value), led:LED3MM
- added R3, R4: (no value), eagle-ltspice:R0204/7
Connections:
- new net DEC+: DEC+.P$1, X1P0.16.S
- new net DEC-: DEC-.P$1, X1P0.14.S
- new net LED3: R3.2, U$1P0.24.S
- new net LED4: R4.2, U$1P0.22.S
- new net N$3: LED3.A, R3.1
- new net N$6: LED4.A, R4.1
- new net RA+: RA+.P$1, X1P0.15.S
- new net RA-: RA-.P$1, X1P0.13.S
- net +3V3: now also UART0.2
- net GND: now also DEC+.P$2, DEC-.P$2, LED3.C, LED4.C, RA+.P$2, RA-.P$2, U$1GND@2.S
Other:
- moved on the sheet: LED2, R2
Changed lines of the file:
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@@
 <part name="GND7" library="supply1" deviceset="GND" device=""/>
 <part name="GND9" library="supply1" deviceset="GND" device=""/>
+<part name="RA+" library="eq-custom2" deviceset="TACT-SWITCH" device=""/>
+<part name="+3V2" library="supply1" deviceset="+3V3" device=""/>
+<part name="GND12" library="supply1" deviceset="GND" device=""/>
+<part name="RA-" library="eq-custom2" deviceset="TACT-SWITCH" device=""/>
+<part name="DEC+" library="eq-custom2" deviceset="TACT-SWITCH" device=""/>
+<part name="DEC-" library="eq-custom2" deviceset="TACT-SWITCH" device=""/>
+<part name="GND13" library="supply1" deviceset="GND" device=""/>
+<part name="GND14" library="supply1" deviceset="GND" device=""/>
+<part name="GND15" library="supply1" deviceset="GND" device=""/>
+<part name="LED3" library="led" deviceset="LED" device="3MM"/>
+<part name="LED4" library="led" deviceset="LED" device="3MM"/>
+<part name="R3" library="eagle-ltspice" deviceset="R" device="0204/7"/>
+<part name="R4" library="eagle-ltspice" deviceset="R" device="0204/7"/>
+<part name="GND16" library="supply1" deviceset="GND" device=""/>
+<part name="GND17" library="supply1" deviceset="GND" device=""/>
+<part name="GND18" library="supply1" deviceset="GND" device=""/>
 </parts>
 <sheets>
@@
 <instance part="GND1" gate="1" x="-152.4" y="10.16"/>
 <instance part="GND2" gate="1" x="-134.62" y="12.7"/>
-<instance part="GND3" gate="1" x="-104.14" y="17.78" rot="R270"/>
+<instance part="GND3" gate="1" x="-104.14" y="25.4" rot="R180"/>
 <instance part="SWD" gate="A" x="-22.86" y="35.56"/>
 <instance part="GND4" gate="1" x="-40.64" y="35.56" rot="R270"/>
@@
 <instance part="C2" gate="G$1" x="-144.78" y="17.78"/>
 <instance part="LED1" gate="G$1" x="-160.02" y="-30.48"/>
-<instance part="LED2" gate="G$1" x="-147.32" y="-30.48"/>
+<instance part="LED2" gate="G$1" x="-149.86" y="-30.48"/>
 <instance part="R1" gate="G$1" x="-160.02" y="-20.32" rot="R90"/>
-<instance part="R2" gate="G$1" x="-147.32" y="-20.32" rot="R90"/>
-<instance part="GND7" gate="1" x="-160.02" y="-43.18"/>
-<instance part="GND9" gate="1" x="-147.32" y="-43.18"/>
+<instance part="R2" gate="G$1" x="-149.86" y="-20.32" rot="R90"/>
+<instance part="GND7" gate="1" x="-160.02" y="-38.1"/>
+<instance part="GND9" gate="1" x="-149.86" y="-38.1"/>
+<instance part="RA+" gate="G$1" x="-177.8" y="-27.94" rot="R270"/>
+<instance part="+3V2" gate="G$1" x="7.62" y="22.86"/>
+<instance part="GND12" gate="1" x="-177.8" y="-43.18"/>
+<instance part="RA-" gate="G$1" x="-190.5" y="-27.94" rot="R270"/>
+<instance part="DEC+" gate="G$1" x="-203.2" y="-27.94" rot="R270"/>
+<instance part="DEC-" gate="G$1" x="-215.9" y="-27.94" rot="R270"/>
+<instance part="GND13" gate="1" x="-190.5" y="-43.18"/>
+<instance part="GND14" gate="1" x="-203.2" y="-43.18"/>
+<instance part="GND15" gate="1" x="-215.9" y="-43.18"/>
+<instance part="LED3" gate="G$1" x="-139.7" y="-30.48"/>
+<instance part="LED4" gate="G$1" x="-129.54" y="-30.48"/>
+<instance part="R3" gate="G$1" x="-139.7" y="-20.32" rot="R90"/>
+<instance part="R4" gate="G$1" x="-129.54" y="-20.32" rot="R90"/>
+<instance part="GND16" gate="1" x="-139.7" y="-38.1"/>
+<instance part="GND17" gate="1" x="-129.54" y="-38.1"/>
+<instance part="GND18" gate="1" x="-83.82" y="5.08" rot="R270"/>
 </instances>
 <busses>
@@
 <pinref part="U$1" gate="GND" pin="S"/>
 <pinref part="GND3" gate="1" pin="GND"/>
+<wire x1="-104.14" y1="22.86" x2="-101.6" y2="17.78" width="0.1524" layer="91"/>
 </segment>
 <segment>
@@
 <segment>
 <pinref part="LED1" gate="G$1" pin="C"/>
-<wire x1="-160.02" y1="-35.56" x2="-160.02" y2="-40.64" width="0.1524" layer="91"/>
 <pinref part="GND7" gate="1" pin="GND"/>
 </segment>
 <segment>
 <pinref part="LED2" gate="G$1" pin="C"/>
-<wire x1="-147.32" y1="-35.56" x2="-147.32" y2="-40.64" width="0.1524" layer="91"/>
 <pinref part="GND9" gate="1" pin="GND"/>
+</segment>
+<segment>
+<pinref part="RA+" gate="G$1" pin="P$2"/>
+<pinref part="GND12" gate="1" pin="GND"/>
+</segment>
+<segment>
+<pinref part="RA-" gate="G$1" pin="P$2"/>
+<pinref part="GND13" gate="1" pin="GND"/>
+</segment>
+<segment>
+<pinref part="DEC+" gate="G$1" pin="P$2"/>
+<pinref part="GND14" gate="1" pin="GND"/>
+</segment>
+<segment>
+<pinref part="DEC-" gate="G$1" pin="P$2"/>
+<pinref part="GND15" gate="1" pin="GND"/>
+</segment>
+<segment>
+<pinref part="LED3" gate="G$1" pin="C"/>
+<pinref part="GND16" gate="1" pin="GND"/>
+</segment>
+<segment>
+<pinref part="LED4" gate="G$1" pin="C"/>
+<pinref part="GND17" gate="1" pin="GND"/>
+</segment>
+<segment>
+<pinref part="U$1" gate="GND@2" pin="S"/>
+<pinref part="GND18" gate="1" pin="GND"/>
 </segment>
 </net>
@@
 <wire x1="15.24" y1="-50.8" x2="15.24" y2="-53.34" width="0.1524" layer="91"/>
 </segment>
+<segment>
+<pinref part="+3V2" gate="G$1" pin="+3V3"/>
+<pinref part="UART0" gate="A" pin="2"/>
+<wire x1="7.62" y1="20.32" x2="7.62" y2="7.62" width="0.1524" layer="91"/>
+<wire x1="7.62" y1="7.62" x2="20.32" y2="7.62" width="0.1524" layer="91"/>
+</segment>
 </net>
 <net name="TX" class="0">
@@
 <pinref part="R2" gate="G$1" pin="1"/>
 <pinref part="LED2" gate="G$1" pin="A"/>
-<wire x1="-147.32" y1="-25.4" x2="-147.32" y2="-27.94" width="0.1524" layer="91"/>
+<wire x1="-149.86" y1="-25.4" x2="-149.86" y2="-27.94" width="0.1524" layer="91"/>
 </segment>
 </net>
@@
 <segment>
 <pinref part="R2" gate="G$1" pin="2"/>
-<wire x1="-147.32" y1="-15.24" x2="-147.32" y2="-10.16" width="0.1524" layer="91"/>
-<label x="-147.32" y="-15.24" size="1.778" layer="95" rot="R90"/>
+<wire x1="-149.86" y1="-15.24" x2="-149.86" y2="-10.16" width="0.1524" layer="91"/>
+<label x="-149.86" y="-15.24" size="1.778" layer="95" rot="R90"/>
 </segment>
 <segment>
@@
 </segment>
 </net>
+<net name="RA+" class="0">
+<segment>
+<pinref part="RA+" gate="G$1" pin="P$1"/>
+<wire x1="-177.8" y1="-15.24" x2="-177.8" y2="-5.08" width="0.1524" layer="91"/>
+<label x="-177.8" y="-10.16" size="1.778" layer="95" rot="R90"/>
+</segment>
+<segment>
+<pinref part="X1" gate="P0.15" pin="S"/>
+<wire x1="-43.18" y1="10.16" x2="-48.26" y2="10.16" width="0.1524" layer="91"/>
+<label x="-48.26" y="10.16" size="1.778" layer="95"/>
+</segment>
+</net>
+<net name="RA-" class="0">
+<segment>
+<pinref part="RA-" gate="G$1" pin="P$1"/>
+<wire x1="-190.5" y1="-15.24" x2="-190.5" y2="-5.08" width="0.1524" layer="91"/>
+<label x="-193.04" y="-5.08" size="1.778" layer="95" rot="R270"/>
+</segment>
+<segment>
+<pinref part="X1" gate="P0.13" pin="S"/>
+<wire x1="-43.18" y1="7.62" x2="-48.26" y2="7.62" width="0.1524" layer="91"/>
+<label x="-48.26" y="7.62" size="1.778" layer="95"/>
+</segment>
+</net>
+<net name="DEC+" class="0">
+<segment>
+<pinref part="DEC+" gate="G$1" pin="P$1"/>
+<wire x1="-203.2" y1="-15.24" x2="-203.2" y2="-5.08" width="0.1524" layer="91"/>
+<label x="-205.74" y="-5.08" size="1.778" layer="95" rot="R270"/>
+</segment>
+<segment>
+<pinref part="X1" gate="P0.16" pin="S"/>
+<wire x1="-22.86" y1="10.16" x2="-27.94" y2="10.16" width="0.1524" layer="91"/>
+<label x="-27.94" y="10.16" size="1.778" layer="95"/>
+</segment>
+</net>
+<net name="DEC-" class="0">
+<segment>
+<pinref part="DEC-" gate="G$1" pin="P$1"/>
+<wire x1="-215.9" y1="-15.24" x2="-215.9" y2="-5.08" width="0.1524" layer="91"/>
+<label x="-218.44" y="-5.08" size="1.778" layer="95" rot="R270"/>
+</segment>
+<segment>
+<pinref part="X1" gate="P0.14" pin="S"/>
+<wire x1="-22.86" y1="7.62" x2="-27.94" y2="7.62" width="0.1524" layer="91"/>
+<label x="-27.94" y="7.62" size="1.778" layer="95"/>
+</segment>
+</net>
+<net name="N$3" class="0">
+<segment>
+<pinref part="LED3" gate="G$1" pin="A"/>
+<pinref part="R3" gate="G$1" pin="1"/>
+<wire x1="-139.7" y1="-25.4" x2="-139.7" y2="-27.94" width="0.1524" layer="91"/>
+</segment>
+</net>
+<net name="N$6" class="0">
+<segment>
+<pinref part="LED4" gate="G$1" pin="A"/>
+<pinref part="R4" gate="G$1" pin="1"/>
+<wire x1="-129.54" y1="-25.4" x2="-129.54" y2="-27.94" width="0.1524" layer="91"/>
+</segment>
+</net>
+<net name="LED3" class="0">
+<segment>
+<pinref part="R3" gate="G$1" pin="2"/>
+<wire x1="-139.7" y1="-15.24" x2="-139.7" y2="-10.16" width="0.1524" layer="91"/>
+<label x="-139.7" y="-15.24" size="1.778" layer="95" rot="R90"/>
+</segment>
+<segment>
+<pinref part="U$1" gate="P0.24" pin="S"/>
+<wire x1="-101.6" y1="12.7" x2="-106.68" y2="12.7" width="0.1524" layer="91"/>
+<label x="-106.68" y="12.7" size="1.778" layer="95"/>
+</segment>
+</net>
+<net name="LED4" class="0">
+<segment>
+<pinref part="R4" gate="G$1" pin="2"/>
+<wire x1="-129.54" y1="-15.24" x2="-129.54" y2="-10.16" width="0.1524" layer="91"/>
+<label x="-129.54" y="-15.24" size="1.778" layer="95" rot="R90"/>
+</segment>
+<segment>
+<pinref part="U$1" gate="P0.22" pin="S"/>
+<wire x1="-101.6" y1="15.24" x2="-106.68" y2="15.24" width="0.1524" layer="91"/>
+<label x="-106.68" y="15.24" size="1.778" layer="95"/>
+</segment>
+</net>

Commit message: board: Change some elements to 	smd
Signed-off-by: Pawel Szewczyk <pfpawelec@gmail.com>
Parts:
- C2: device rcl:CPOL-EUE2.5-6 -> rcl:CPOL-EUSMCC
- LED1, LED2, LED3, LED4: device led:LED3MM -> led:LEDSML1206
- R1, R2, R3, R4: device eagle-ltspice:R0204/7 -> eagle-ltspice:RR1206
Changed lines of the file:
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@@
 <grid distance="0.1" unitdist="inch" unit="inch" style="lines" multiple="1" display="no" altdistance="0.01" altunitdist="inch" altunit="inch"/>
 <layers>
-<layer number="1" name="Top" color="4" fill="10" visible="no" active="no"/>
-<layer number="16" name="Bottom" color="1" fill="1" visible="no" active="no"/>
-<layer number="17" name="Pads" color="2" fill="1" visible="no" active="no"/>
-<layer number="18" name="Vias" color="2" fill="1" visible="no" active="no"/>
-<layer number="19" name="Unrouted" color="6" fill="1" visible="no" active="no"/>
-<layer number="20" name="Dimension" color="15" fill="1" visible="no" active="no"/>
-<layer number="21" name="tPlace" color="7" fill="1" visible="no" active="no"/>
-<layer number="22" name="bPlace" color="7" fill="1" visible="no" active="no"/>
-<layer number="23" name="tOrigins" color="15" fill="1" visible="no" active="no"/>
-<layer number="24" name="bOrigins" color="15" fill="1" visible="no" active="no"/>
-<layer number="25" name="tNames" color="7" fill="1" visible="no" active="no"/>
-<layer number="26" name="bNames" color="7" fill="1" visible="no" active="no"/>
-<layer number="27" name="tValues" color="7" fill="1" visible="no" active="no"/>
-<layer number="28" name="bValues" color="7" fill="1" visible="no" active="no"/>
+<layer number="1" name="Top" color="4" fill="1" visible="yes" active="no"/>
+<layer number="16" name="Bottom" color="1" fill="1" visible="yes" active="no"/>
+<layer number="17" name="Pads" color="2" fill="1" visible="yes" active="no"/>
+<layer number="18" name="Vias" color="2" fill="1" visible="yes" active="no"/>
+<layer number="19" name="Unrouted" color="6" fill="1" visible="yes" active="no"/>
+<layer number="20" name="Dimension" color="15" fill="1" visible="yes" active="no"/>
+<layer number="21" name="tPlace" color="7" fill="1" visible="yes" active="no"/>
+<layer number="22" name="bPlace" color="7" fill="1" visible="yes" active="no"/>
+<layer number="23" name="tOrigins" color="15" fill="1" visible="yes" active="no"/>
+<layer number="24" name="bOrigins" color="15" fill="1" visible="yes" active="no"/>
+<layer number="25" name="tNames" color="7" fill="1" visible="yes" active="no"/>
+<layer number="26" name="bNames" color="7" fill="1" visible="yes" active="no"/>
+<layer number="27" name="tValues" color="7" fill="1" visible="yes" active="no"/>
+<layer number="28" name="bValues" color="7" fill="1" visible="yes" active="no"/>
 <layer number="29" name="tStop" color="7" fill="3" visible="no" active="no"/>
 <layer number="30" name="bStop" color="7" fill="6" visible="no" active="no"/>
@@
 <layer number="35" name="tGlue" color="7" fill="4" visible="no" active="no"/>
 <layer number="36" name="bGlue" color="7" fill="5" visible="no" active="no"/>
-<layer number="37" name="tTest" color="7" fill="1" visible="no" active="no"/>
-<layer number="38" name="bTest" color="7" fill="1" visible="no" active="no"/>
+<layer number="37" name="tTest" color="7" fill="1" visible="yes" active="no"/>
+<layer number="38" name="bTest" color="7" fill="1" visible="yes" active="no"/>
 <layer number="39" name="tKeepout" color="4" fill="11" visible="no" active="no"/>
 <layer number="40" name="bKeepout" color="1" fill="11" visible="no" active="no"/>
@@
 <layer number="44" name="Drills" color="7" fill="1" visible="no" active="no"/>
 <layer number="45" name="Holes" color="7" fill="1" visible="no" active="no"/>
-<layer number="46" name="Milling" color="3" fill="1" visible="no" active="no"/>
-<layer number="47" name="Measures" color="7" fill="1" visible="no" active="no"/>
-<layer number="48" name="Document" color="7" fill="1" visible="no" active="no"/>
-<layer number="49" name="Reference" color="7" fill="1" visible="no" active="no"/>
-<layer number="50" name="dxf" color="7" fill="1" visible="no" active="no"/>
-<layer number="51" name="tDocu" color="26" fill="1" visible="no" active="no"/>
-<layer number="52" name="bDocu" color="7" fill="1" visible="no" active="no"/>
-<layer number="53" name="tGND_GNDA" color="7" fill="1" visible="no" active="no"/>
-<layer number="54" name="bGND_GNDA" color="7" fill="1" visible="no" active="no"/>
-<layer number="56" name="wert" color="7" fill="1" visible="no" active="no"/>
-<layer number="57" name="tCAD" color="7" fill="1" visible="no" active="no"/>
+<layer number="46" name="Milling" color="3" fill="1" visible="yes" active="no"/>
+<layer number="47" name="Measures" color="7" fill="1" visible="yes" active="no"/>
+<layer number="48" name="Document" color="7" fill="1" visible="yes" active="no"/>
+<layer number="49" name="Reference" color="7" fill="1" visible="yes" active="no"/>
+<layer number="50" name="dxf" color="7" fill="1" visible="yes" active="no"/>
+<layer number="51" name="tDocu" color="7" fill="1" visible="yes" active="no"/>
+<layer number="52" name="bDocu" color="7" fill="1" visible="yes" active="no"/>
+<layer number="53" name="tGND_GNDA" color="7" fill="1" visible="yes" active="no"/>
+<layer number="54" name="bGND_GNDA" color="7" fill="1" visible="yes" active="no"/>
+<layer number="56" name="wert" color="7" fill="1" visible="yes" active="no"/>
+<layer number="57" name="tCAD" color="7" fill="1" visible="yes" active="no"/>
 <layer number="90" name="Modules" color="5" fill="1" visible="yes" active="yes"/>
 <layer number="91" name="Nets" color="2" fill="1" visible="yes" active="yes"/>
@@
 <part name="MOT-DEC" library="con-ptr500" deviceset="AK500/4" device=""/>
 <part name="IC2" library="lf33" deviceset="LFXXCV" device="S"/>
-<part name="C2" library="rcl" deviceset="CPOL-EU" device="E2.5-6"/>
-<part name="LED1" library="led" deviceset="LED" device="3MM"/>
-<part name="LED2" library="led" deviceset="LED" device="3MM"/>
-<part name="R1" library="eagle-ltspice" deviceset="R" device="0204/7"/>
-<part name="R2" library="eagle-ltspice" deviceset="R" device="0204/7"/>
+<part name="C2" library="rcl" deviceset="CPOL-EU" device="SMCC"/>
+<part name="LED1" library="led" deviceset="LED" device="SML1206"/>
+<part name="LED2" library="led" deviceset="LED" device="SML1206"/>
+<part name="R1" library="eagle-ltspice" deviceset="R" device="R1206"/>
+<part name="R2" library="eagle-ltspice" deviceset="R" device="R1206"/>
 <part name="GND7" library="supply1" deviceset="GND" device=""/>
 <part name="GND9" library="supply1" deviceset="GND" device=""/>
@@
 <part name="GND14" library="supply1" deviceset="GND" device=""/>
 <part name="GND15" library="supply1" deviceset="GND" device=""/>
-<part name="LED3" library="led" deviceset="LED" device="3MM"/>
-<part name="LED4" library="led" deviceset="LED" device="3MM"/>
-<part name="R3" library="eagle-ltspice" deviceset="R" device="0204/7"/>
-<part name="R4" library="eagle-ltspice" deviceset="R" device="0204/7"/>
+<part name="LED3" library="led" deviceset="LED" device="SML1206"/>
+<part name="LED4" library="led" deviceset="LED" device="SML1206"/>
+<part name="R3" library="eagle-ltspice" deviceset="R" device="R1206"/>
+<part name="R4" library="eagle-ltspice" deviceset="R" device="R1206"/>
 <part name="GND16" library="supply1" deviceset="GND" device=""/>
 <part name="GND17" library="supply1" deviceset="GND" device=""/>

Commit message: Change more elements to smd
Signed-off-by: Pawel Szewczyk <pfpawelec@gmail.com>
Parts:
- removed IC2: (no value), lf33:LFXXCVS
- added IC1: REG1117, burr-brown:REG1117
Connections:
- net +12V: now also IC1.VIN; no longer IC2.IN
- net +3V3: now also IC1.VOUT; no longer IC2.OUT
- net GND: now also IC1.GND; no longer IC2.GND
Other:
- moved on the sheet: C2, J1
Changed lines of the file:
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@@
 <part name="MOT-RA" library="con-ptr500" deviceset="AK500/4" device=""/>
 <part name="MOT-DEC" library="con-ptr500" deviceset="AK500/4" device=""/>
-<part name="IC2" library="lf33" deviceset="LFXXCV" device="S"/>
 <part name="C2" library="rcl" deviceset="CPOL-EU" device="SMCC"/>
 <part name="LED1" library="led" deviceset="LED" device="SML1206"/>
@@
 <part name="GND17" library="supply1" deviceset="GND" device=""/>
 <part name="GND18" library="supply1" deviceset="GND" device=""/>
+<part name="IC1" library="burr-brown" deviceset="REG1117" device=""/>
 </parts>
 <sheets>
@@
 <instance part="X1" gate="SWD" x="-20.32" y="12.7"/>
 <instance part="X1" gate="SWDIO" x="-40.64" y="12.7"/>
-<instance part="J1" gate="G$1" x="-162.56" y="20.32"/>
-<instance part="GND1" gate="1" x="-152.4" y="10.16"/>
-<instance part="GND2" gate="1" x="-134.62" y="12.7"/>
+<instance part="J1" gate="G$1" x="-175.26" y="20.32"/>
+<instance part="GND1" gate="1" x="-165.1" y="10.16"/>
+<instance part="GND2" gate="1" x="-139.7" y="2.54"/>
 <instance part="GND3" gate="1" x="-104.14" y="25.4" rot="R180"/>
 <instance part="SWD" gate="A" x="-22.86" y="35.56"/>
 <instance part="GND4" gate="1" x="-40.64" y="35.56" rot="R270"/>
 <instance part="UART0" gate="A" x="22.86" y="2.54"/>
-<instance part="P+1" gate="1" x="-149.86" y="33.02"/>
+<instance part="P+1" gate="1" x="-162.56" y="33.02"/>
 <instance part="+3V1" gate="G$1" x="-114.3" y="35.56"/>
 <instance part="GND5" gate="1" x="15.24" y="25.4" rot="R180"/>
@@
 <instance part="MOT-DEC" gate="-3" x="-43.18" y="-78.74" rot="R90"/>
 <instance part="MOT-DEC" gate="-4" x="-38.1" y="-78.74" rot="R90"/>
-<instance part="IC2" gate="A" x="-134.62" y="22.86"/>
-<instance part="C2" gate="G$1" x="-144.78" y="17.78"/>
+<instance part="C2" gate="G$1" x="-157.48" y="17.78"/>
 <instance part="LED1" gate="G$1" x="-160.02" y="-30.48"/>
 <instance part="LED2" gate="G$1" x="-149.86" y="-30.48"/>
@@
 <instance part="GND17" gate="1" x="-129.54" y="-38.1"/>
 <instance part="GND18" gate="1" x="-83.82" y="5.08" rot="R270"/>
+<instance part="IC1" gate="G$1" x="-139.7" y="22.86"/>
 </instances>
 <busses>
@@
 <pinref part="J1" gate="G$1" pin="2"/>
 <pinref part="GND1" gate="1" pin="GND"/>
-<wire x1="-154.94" y1="20.32" x2="-152.4" y2="20.32" width="0.1524" layer="91"/>
-<wire x1="-152.4" y1="20.32" x2="-152.4" y2="12.7" width="0.1524" layer="91"/>
+<wire x1="-167.64" y1="20.32" x2="-165.1" y2="20.32" width="0.1524" layer="91"/>
+<wire x1="-165.1" y1="20.32" x2="-165.1" y2="12.7" width="0.1524" layer="91"/>
 <pinref part="J1" gate="G$1" pin="3"/>
-<wire x1="-154.94" y1="17.78" x2="-152.4" y2="17.78" width="0.1524" layer="91"/>
-<wire x1="-152.4" y1="17.78" x2="-152.4" y2="12.7" width="0.1524" layer="91"/>
-<wire x1="-144.78" y1="12.7" x2="-152.4" y2="12.7" width="0.1524" layer="91"/>
+<wire x1="-167.64" y1="17.78" x2="-165.1" y2="17.78" width="0.1524" layer="91"/>
+<wire x1="-165.1" y1="17.78" x2="-165.1" y2="12.7" width="0.1524" layer="91"/>
+<wire x1="-157.48" y1="12.7" x2="-165.1" y2="12.7" width="0.1524" layer="91"/>
 <pinref part="C2" gate="G$1" pin="-"/>
 </segment>
@@
 </segment>
 <segment>
-<pinref part="IC2" gate="A" pin="GND"/>
-<pinref part="GND2" gate="1" pin="GND"/>
-</segment>
-<segment>
 <pinref part="LED1" gate="G$1" pin="C"/>
 <pinref part="GND7" gate="1" pin="GND"/>
@@
 <pinref part="GND18" gate="1" pin="GND"/>
 </segment>
+<segment>
+<pinref part="IC1" gate="G$1" pin="GND"/>
+<pinref part="GND2" gate="1" pin="GND"/>
+<wire x1="-139.7" y1="10.16" x2="-139.7" y2="5.08" width="0.1524" layer="91"/>
+</segment>
 </net>
 <net name="+12V" class="0">
 <segment>
 <pinref part="J1" gate="G$1" pin="1"/>
-<wire x1="-154.94" y1="22.86" x2="-149.86" y2="22.86" width="0.1524" layer="91"/>
-<wire x1="-149.86" y1="22.86" x2="-144.78" y2="22.86" width="0.1524" layer="91"/>
-<junction x="-149.86" y="22.86"/>
+<wire x1="-167.64" y1="22.86" x2="-162.56" y2="22.86" width="0.1524" layer="91"/>
+<wire x1="-162.56" y1="22.86" x2="-157.48" y2="22.86" width="0.1524" layer="91"/>
+<junction x="-162.56" y="22.86"/>
 <pinref part="P+1" gate="1" pin="+12V"/>
-<wire x1="-144.78" y1="22.86" x2="-142.24" y2="22.86" width="0.1524" layer="91"/>
-<wire x1="-149.86" y1="22.86" x2="-149.86" y2="30.48" width="0.1524" layer="91"/>
-<pinref part="IC2" gate="A" pin="IN"/>
-<wire x1="-144.78" y1="20.32" x2="-144.78" y2="22.86" width="0.1524" layer="91"/>
+<wire x1="-157.48" y1="22.86" x2="-154.94" y2="22.86" width="0.1524" layer="91"/>
+<wire x1="-162.56" y1="22.86" x2="-162.56" y2="30.48" width="0.1524" layer="91"/>
+<wire x1="-157.48" y1="20.32" x2="-157.48" y2="22.86" width="0.1524" layer="91"/>
 <pinref part="C2" gate="G$1" pin="+"/>
+<pinref part="IC1" gate="G$1" pin="VIN"/>
+<wire x1="-152.4" y1="22.86" x2="-154.94" y2="22.86" width="0.1524" layer="91"/>
 </segment>
 <segment>
@@
 <wire x1="-114.3" y1="33.02" x2="-114.3" y2="22.86" width="0.1524" layer="91"/>
 <junction x="-114.3" y="22.86"/>
-<pinref part="IC2" gate="A" pin="OUT"/>
 <wire x1="-127" y1="22.86" x2="-114.3" y2="22.86" width="0.1524" layer="91"/>
-</segment>
-<segment>
+<pinref part="IC1" gate="G$1" pin="VOUT"/>
+</segment>
+<segment>
