File: eagle/proto.sch (EAGLE design)
At the start: 23 parts, among them IC1 REG1117, J1 DCJ0202, X1 NRF51822-RIGHT

Commit message: eagle: Add ST4 port
Signed-off-by: Pawel Szewczyk <pfpawelec@gmail.com>
Parts:
- removed LED4: (no value), led:LEDSML1206
- removed R4: (no value), eagle-ltspice:RR1206
- added ST4: RJ11, SparkFun-Connectors:RJ11-6
Connections:
- removed net LED4: R4.2, U$1P0.22.S
- removed net N$6: LED4.A, R4.1
- net DEC+: now also ST4.4
- net DEC-: now also ST4.5
- net GND: now also ST4.2; no longer LED4.C
- net LED2: now also U$1P0.24.S; no longer U$1P0.26.S
- net LED3: now also U$1P0.22.S; no longer U$1P0.24.S
- net RA+: now also ST4.3
- net RA-: now also ST4.6
Changed lines of the file:
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@@
 <layer number="56" name="wert" color="7" fill="1" visible="yes" active="no"/>
 <layer number="57" name="tCAD" color="7" fill="1" visible="yes" active="no"/>
+<layer number="59" name="tCarbon" color="7" fill="1" visible="no" active="no"/>
+<layer number="60" name="bCarbon" color="7" fill="1" visible="no" active="no"/>
 <layer number="90" name="Modules" color="5" fill="1" visible="yes" active="yes"/>
 <layer number="91" name="Nets" color="2" fill="1" visible="yes" active="yes"/>
@@
 <layer number="112" name="tSilk" color="7" fill="1" visible="yes" active="yes"/>
 <layer number="113" name="IDFDebug" color="7" fill="1" visible="yes" active="yes"/>
+<layer number="114" name="Badge_Outline" color="7" fill="1" visible="yes" active="yes"/>
+<layer number="115" name="ReferenceISLANDS" color="7" fill="1" visible="yes" active="yes"/>
 <layer number="116" name="Patch_BOT" color="7" fill="1" visible="yes" active="yes"/>
+<layer number="118" name="Rect_Pads" color="7" fill="1" visible="yes" active="yes"/>
 <layer number="121" name="_tsilk" color="7" fill="1" visible="yes" active="yes"/>
 <layer number="122" name="_bsilk" color="7" fill="1" visible="yes" active="yes"/>
@@
 <layer number="127" name="_tValues" color="7" fill="1" visible="yes" active="yes"/>
 <layer number="128" name="_bValues" color="7" fill="1" visible="yes" active="yes"/>
+<layer number="129" name="Mask" color="7" fill="1" visible="yes" active="yes"/>
 <layer number="131" name="tAdjust" color="7" fill="1" visible="yes" active="yes"/>
 <layer number="132" name="bAdjust" color="7" fill="1" visible="yes" active="yes"/>
@@
 <layer number="223" name="223bmp" color="7" fill="1" visible="yes" active="yes"/>
 <layer number="224" name="224bmp" color="7" fill="1" visible="yes" active="yes"/>
+<layer number="225" name="225bmp" color="7" fill="1" visible="yes" active="yes"/>
+<layer number="226" name="226bmp" color="7" fill="1" visible="yes" active="yes"/>
+<layer number="227" name="227bmp" color="7" fill="1" visible="yes" active="yes"/>
+<layer number="228" name="228bmp" color="7" fill="1" visible="yes" active="yes"/>
+<layer number="229" name="229bmp" color="7" fill="1" visible="yes" active="yes"/>
+<layer number="230" name="230bmp" color="7" fill="1" visible="yes" active="yes"/>
+<layer number="231" name="231bmp" color="7" fill="1" visible="yes" active="yes"/>
+<layer number="232" name="Eagle3D_PG2" color="7" fill="1" visible="yes" active="yes"/>
+<layer number="233" name="Eagle3D_PG3" color="7" fill="1" visible="yes" active="yes"/>
 <layer number="248" name="Housing" color="7" fill="1" visible="yes" active="yes"/>
 <layer number="249" name="Edge" color="7" fill="1" visible="yes" active="yes"/>
@@
 <layer number="251" name="SMDround" color="7" fill="1" visible="yes" active="yes"/>
 <layer number="254" name="cooling" color="7" fill="1" visible="yes" active="yes"/>
+<layer number="255" name="routoute" color="7" fill="1" visible="yes" active="yes"/>
 </layers>
 <schematic xreflabel="%F%N/%S.%C%R" xrefpart="/%S.%C%R">
@@
 <part name="GND15" library="supply1" deviceset="GND" device=""/>
 <part name="LED3" library="led" deviceset="LED" device="SML1206"/>
-<part name="LED4" library="led" deviceset="LED" device="SML1206"/>
 <part name="R3" library="eagle-ltspice" deviceset="R" device="R1206"/>
-<part name="R4" library="eagle-ltspice" deviceset="R" device="R1206"/>
 <part name="GND16" library="supply1" deviceset="GND" device=""/>
-<part name="GND17" library="supply1" deviceset="GND" device=""/>
 <part name="GND18" library="supply1" deviceset="GND" device=""/>
 <part name="IC1" library="burr-brown" deviceset="REG1117" device=""/>
+<part name="ST4" library="SparkFun-Connectors" deviceset="RJ11-6" device="" value="RJ11"/>
+<part name="GND17" library="supply1" deviceset="GND" device=""/>
 </parts>
 <sheets>
@@
 <instance part="GND15" gate="1" x="-215.9" y="-43.18"/>
 <instance part="LED3" gate="G$1" x="-139.7" y="-30.48"/>
-<instance part="LED4" gate="G$1" x="-129.54" y="-30.48"/>
 <instance part="R3" gate="G$1" x="-139.7" y="-20.32" rot="R90"/>
-<instance part="R4" gate="G$1" x="-129.54" y="-20.32" rot="R90"/>
 <instance part="GND16" gate="1" x="-139.7" y="-38.1"/>
-<instance part="GND17" gate="1" x="-129.54" y="-38.1"/>
 <instance part="GND18" gate="1" x="-83.82" y="5.08" rot="R270"/>
 <instance part="IC1" gate="G$1" x="-139.7" y="22.86"/>
+<instance part="ST4" gate="G$1" x="-73.66" y="35.56" rot="R270"/>
+<instance part="GND17" gate="1" x="-78.74" y="25.4"/>
 </instances>
 <busses>
@@
 </segment>
 <segment>
-<pinref part="LED4" gate="G$1" pin="C"/>
-<pinref part="GND17" gate="1" pin="GND"/>
-</segment>
-<segment>
 <pinref part="U$1" gate="GND@2" pin="S"/>
 <pinref part="GND18" gate="1" pin="GND"/>
@@
 <pinref part="GND2" gate="1" pin="GND"/>
 <wire x1="-139.7" y1="10.16" x2="-139.7" y2="5.08" width="0.1524" layer="91"/>
+</segment>
+<segment>
+<pinref part="GND17" gate="1" pin="GND"/>
+<pinref part="ST4" gate="G$1" pin="2"/>
+<wire x1="-78.74" y1="27.94" x2="-76.2" y2="27.94" width="0.1524" layer="91"/>
+<wire x1="-76.2" y1="27.94" x2="-76.2" y2="30.48" width="0.1524" layer="91"/>
 </segment>
 </net>
@@
 </segment>
 <segment>
-<pinref part="U$1" gate="P0.26" pin="S"/>
-<wire x1="-101.6" y1="10.16" x2="-106.68" y2="10.16" width="0.1524" layer="91"/>
-<label x="-106.68" y="10.16" size="1.778" layer="95"/>
+<pinref part="U$1" gate="P0.24" pin="S"/>
+<wire x1="-101.6" y1="12.7" x2="-106.68" y2="12.7" width="0.1524" layer="91"/>
+<label x="-106.68" y="12.7" size="1.778" layer="95"/>
 </segment>
 </net>
@@
 <label x="-48.26" y="10.16" size="1.778" layer="95"/>
 </segment>
+<segment>
+<pinref part="ST4" gate="G$1" pin="3"/>
+<wire x1="-73.66" y1="30.48" x2="-73.66" y2="25.4" width="0.1524" layer="91"/>
+<label x="-73.66" y="25.4" size="1.778" layer="95" rot="R90"/>
+</segment>
 </net>
 <net name="RA-" class="0">
@@
 <label x="-48.26" y="7.62" size="1.778" layer="95"/>
 </segment>
+<segment>
+<pinref part="ST4" gate="G$1" pin="6"/>
+<wire x1="-66.04" y1="30.48" x2="-66.04" y2="25.4" width="0.1524" layer="91"/>
+<label x="-66.04" y="25.4" size="1.778" layer="95" rot="R90"/>
+</segment>
 </net>
 <net name="DEC+" class="0">
@@
 <label x="-27.94" y="10.16" size="1.778" layer="95"/>
 </segment>
+<segment>
+<pinref part="ST4" gate="G$1" pin="4"/>
+<wire x1="-71.12" y1="30.48" x2="-71.12" y2="25.4" width="0.1524" layer="91"/>
+<label x="-71.12" y="25.4" size="1.778" layer="95" rot="R90"/>
+</segment>
 </net>
 <net name="DEC-" class="0">
@@
 <label x="-27.94" y="7.62" size="1.778" layer="95"/>
 </segment>
+<segment>
+<pinref part="ST4" gate="G$1" pin="5"/>
+<wire x1="-68.58" y1="30.48" x2="-68.58" y2="25.4" width="0.1524" layer="91"/>
+<label x="-68.58" y="25.4" size="1.778" layer="95" rot="R90"/>
+</segment>
 </net>
 <net name="N$3" class="0">
@@
 </segment>
 </net>
-<net name="N$6" class="0">
-<segment>
-<pinref part="LED4" gate="G$1" pin="A"/>
-<pinref part="R4" gate="G$1" pin="1"/>
-<wire x1="-129.54" y1="-25.4" x2="-129.54" y2="-27.94" width="0.1524" layer="91"/>
-</segment>
-</net>
 <net name="LED3" class="0">
 <segment>
@@
 </segment>
 <segment>
-<pinref part="U$1" gate="P0.24" pin="S"/>
-<wire x1="-101.6" y1="12.7" x2="-106.68" y2="12.7" width="0.1524" layer="91"/>
-<label x="-106.68" y="12.7" size="1.778" layer="95"/>
-</segment>
-</net>
-<net name="LED4" class="0">
-<segment>
-<pinref part="R4" gate="G$1" pin="2"/>
-<wire x1="-129.54" y1="-15.24" x2="-129.54" y2="-10.16" width="0.1524" layer="91"/>
-<label x="-129.54" y="-15.24" size="1.778" layer="95" rot="R90"/>
-</segment>
-<segment>
